File: Schematics/TinyPico-Cycling-Tracker/Bottom_board.kicad_sch (KiCad schematic)
At the start: 3 parts, among them U10 MicroSD Card Adapter, U8 TinyPico, U9 GPS6MV2

Commit message: fix: move physical pin to the schematic
Parts:
- renumbered U10 to U1, U8 to U2, U9 to U3
Connections:
- net SW_TP: now also U2.8 (IO33); no longer U2.16 (IO4)

Commit message: chore: position of Push Button & Mounting Holes
Parts:
- added H1, H2, H3, H4: MountingHole, MountingHole:MountingHole_3mm, symbol Mechanical:MountingHole
- renumbered U1 to U10, U2 to U8, U3 to U9

Commit message: chore: INT in schematic and PCB
Connections:
- net INT: now reaches U8.13 (IO27)
- no-connect marks 7 -> 6
Changed lines of the file:
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@@
-	)
-	(no_connect
-		(at 149.86 87.63)
 	)
 	(no_connect
@@
 		(pts
 			(xy 157.48 92.71) (xy 157.48 85.09)
+		)
+		(stroke
+			(width 0)
+			(type default)
+		)
+	)
+	(wire
+		(pts
+			(xy 149.86 87.63) (xy 152.4 87.63)
 		)
 		(stroke
@@
 			)
 			(justify right)
+		)
+	)
+	(hierarchical_label "INT"
+		(shape input)
+		(at 152.4 87.63 0)
+		(effects
+			(font
+				(size 1.27 1.27)
+			)
+			(justify left)
 		)
 	)
@@
 		)
 		(instances
-			(project ""
+			(project "TinyPico-Cycling-Tracker"
 				(path "/c19b4b11-d562-4619-8198-7fbe4f513d32/a53ff72c-e30f-413f-a95e-3ac33687ad4a"
 					(reference "H2")
@@
 				)
 			)
-			(project ""
+			(project "TinyPico-Cycling-Tracker"
 				(path "/c19b4b11-d562-4619-8198-7fbe4f513d32/a53ff72c-e30f-413f-a95e-3ac33687ad4a"
 					(reference "U9")
@@
 				)
 			)
-			(project ""
+			(project "TinyPico-Cycling-Tracker"
 				(path "/c19b4b11-d562-4619-8198-7fbe4f513d32/a53ff72c-e30f-413f-a95e-3ac33687ad4a"
 					(reference "#FLG02")
@@
 				)
 			)
-			(project ""
+			(project "TinyPico-Cycling-Tracker"
 				(path "/c19b4b11-d562-4619-8198-7fbe4f513d32/a53ff72c-e30f-413f-a95e-3ac33687ad4a"
 					(reference "U8")
@@
 				)
 			)
-			(project ""
+			(project "TinyPico-Cycling-Tracker"
 				(path "/c19b4b11-d562-4619-8198-7fbe4f513d32/a53ff72c-e30f-413f-a95e-3ac33687ad4a"
 					(reference "#PWR07")
@@
 				)
 			)
-			(project ""
+			(project "TinyPico-Cycling-Tracker"
 				(path "/c19b4b11-d562-4619-8198-7fbe4f513d32/a53ff72c-e30f-413f-a95e-3ac33687ad4a"
 					(reference "U10")
@@
 				)
 			)
-			(project ""
+			(project "TinyPico-Cycling-Tracker"
 				(path "/c19b4b11-d562-4619-8198-7fbe4f513d32/a53ff72c-e30f-413f-a95e-3ac33687ad4a"
 					(reference "#PWR08")
@@
 		)
 		(instances
-			(project ""
+			(project "TinyPico-Cycling-Tracker"
 				(path "/c19b4b11-d562-4619-8198-7fbe4f513d32/a53ff72c-e30f-413f-a95e-3ac33687ad4a"
 					(reference "H1")
