File: Schematics/TinyPico-Cycling-Tracker/Upper_board.kicad_sch (KiCad schematic)
At the start: 4 parts, among them SW2 SW_Push, U6 module_mpu6050, U7 SSD1306 0.96" OLED

Commit message: chore: update PCB to recude the vias
Parts:
- SW?: renamed from SW2; footprint Button_Switch_THT:SW_TH_Tactile_Omron_B3F-102x -> SPST_Button:SPST_Button
- renumbered R2 to R?, U6 to U?, U7 to U?
Changed lines of the file:
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@@
 		(dnp no)
 		(fields_autoplaced yes)
-		(property "Reference" "#FLG03"
+		(property "Reference" "#FLG?"
 			(at 161.29 45.085 0)
 			(effects
@@
 		)
 		(instances
+			(project "Upper_board"
+				(path "/437a6128-0e45-45ff-808b-ce6204aa4772"
+					(reference "#FLG?")
+					(unit 1)
+				)
+			)
 			(project ""
 				(path "/c19b4b11-d562-4619-8198-7fbe4f513d32/087e4c3f-dadb-4b00-b947-e0c7adeb7ff5"
@@
 		(dnp no)
 		(fields_autoplaced yes)
-		(property "Reference" "SW2"
+		(property "Reference" "SW?"
 			(at 162.56 72.3899 90)
 			(effects
@@
 			)
 		)
-		(property "Footprint" "Button_Switch_THT:SW_TH_Tactile_Omron_B3F-102x"
+		(property "Footprint" "SPST_Button:SPST_Button"
 			(at 156.21 73.66 0)
 			(effects
@@
 		)
 		(instances
+			(project "Upper_board"
+				(path "/437a6128-0e45-45ff-808b-ce6204aa4772"
+					(reference "SW?")
+					(unit 1)
+				)
+			)
 			(project ""
 				(path "/c19b4b11-d562-4619-8198-7fbe4f513d32/087e4c3f-dadb-4b00-b947-e0c7adeb7ff5"
@@
 		(dnp no)
 		(fields_autoplaced yes)
-		(property "Reference" "#PWR01"
+		(property "Reference" "#PWR?"
 			(at 168.91 50.8 0)
 			(effects
@@
 		)
 		(instances
+			(project "Upper_board"
+				(path "/437a6128-0e45-45ff-808b-ce6204aa4772"
+					(reference "#PWR?")
+					(unit 1)
+				)
+			)
 			(project ""
 				(path "/c19b4b11-d562-4619-8198-7fbe4f513d32/087e4c3f-dadb-4b00-b947-e0c7adeb7ff5"
@@
 		(dnp no)
 		(fields_autoplaced yes)
-		(property "Reference" "U6"
+		(property "Reference" "U?"
 			(at 199.39 72.3899 0)
 			(effects
@@
 		)
 		(instances
+			(project "Upper_board"
+				(path "/437a6128-0e45-45ff-808b-ce6204aa4772"
+					(reference "U?")
+					(unit 1)
+				)
+			)
 			(project ""
 				(path "/c19b4b11-d562-4619-8198-7fbe4f513d32/087e4c3f-dadb-4b00-b947-e0c7adeb7ff5"
@@
 		(dnp no)
 		(fields_autoplaced yes)
-		(property "Reference" "U7"
+		(property "Reference" "U?"
 			(at 193.04 50.1649 0)
 			(effects
@@
 		)
 		(instances
+			(project "Upper_board"
+				(path "/437a6128-0e45-45ff-808b-ce6204aa4772"
+					(reference "U?")
+					(unit 1)
+				)
+			)
 			(project ""
 				(path "/c19b4b11-d562-4619-8198-7fbe4f513d32/087e4c3f-dadb-4b00-b947-e0c7adeb7ff5"
@@
 		(dnp no)
 		(fields_autoplaced yes)
-		(property "Reference" "R2"
+		(property "Reference" "R?"
 			(at 163.83 57.1499 0)
 			(effects
@@
 		)
 		(instances
+			(project "Upper_board"
+				(path "/437a6128-0e45-45ff-808b-ce6204aa4772"
+					(reference "R?")
+					(unit 1)
+				)
+			)
 			(project ""
 				(path "/c19b4b11-d562-4619-8198-7fbe4f513d32/087e4c3f-dadb-4b00-b947-e0c7adeb7ff5"
@@
 		(dnp no)
 		(fields_autoplaced yes)
-		(property "Reference" "#PWR06"
+		(property "Reference" "#PWR?"
 			(at 168.91 97.79 0)
 			(effects
@@
 		)
 		(instances
+			(project "Upper_board"
+				(path "/437a6128-0e45-45ff-808b-ce6204aa4772"
+					(reference "#PWR?")
+					(unit 1)
+				)
+			)
 			(project ""
 				(path "/c19b4b11-d562-4619-8198-7fbe4f513d32/087e4c3f-dadb-4b00-b947-e0c7adeb7ff5"
@@
 		(dnp no)
 		(fields_autoplaced yes)
-		(property "Reference" "#FLG01"
+		(property "Reference" "#FLG?"
 			(at 212.09 80.645 0)
 			(effects
@@
 		)
 		(instances
+			(project "Upper_board"
+				(path "/437a6128-0e45-45ff-808b-ce6204aa4772"
+					(reference "#FLG?")
+					(unit 1)
+				)
+			)
 			(project ""
 				(path "/c19b4b11-d562-4619-8198-7fbe4f513d32/087e4c3f-dadb-4b00-b947-e0c7adeb7ff5"
@@
 		)
 	)
+	(sheet_instances
+		(path "/"
+			(page "1")
+		)
+	)
+	(embedded_fonts no)
 )

Commit message: chore: position of Push Button & Mounting Holes
Parts:
- added H5, H6, H7, H8: MountingHole, MountingHole:MountingHole_3mm, symbol Mechanical:MountingHole
- gave numbers to parts that had none: 4

Commit message: chore: INT in schematic and PCB
Connections:
- net INT: now reaches U6.8 (INT)
- no-connect marks 4 -> 3
Changed lines of the file:
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@@
 		(at 179.07 80.01)
 	)
-	(no_connect
-		(at 179.07 82.55)
-	)
 	(wire
 		(pts
@@
 		(pts
 			(xy 179.07 46.99) (xy 176.53 46.99)
+		)
+		(stroke
+			(width 0)
+			(type default)
+		)
+	)
+	(wire
+		(pts
+			(xy 176.53 82.55) (xy 179.07 82.55)
 		)
 		(stroke
@@
 			)
 			(justify left)
+		)
+	)
+	(hierarchical_label "INT"
+		(shape input)
+		(at 176.53 82.55 180)
+		(effects
+			(font
+				(size 1.27 1.27)
+			)
+			(justify right)
 		)
 	)
@@
 				)
 			)
-			(project ""
+			(project "TinyPico-Cycling-Tracker"
 				(path "/c19b4b11-d562-4619-8198-7fbe4f513d32/087e4c3f-dadb-4b00-b947-e0c7adeb7ff5"
 					(reference "#FLG03")
@@
 				)
 			)
-			(project ""
+			(project "TinyPico-Cycling-Tracker"
 				(path "/c19b4b11-d562-4619-8198-7fbe4f513d32/087e4c3f-dadb-4b00-b947-e0c7adeb7ff5"
 					(reference "SW2")
@@
 				)
 			)
-			(project ""
+			(project "TinyPico-Cycling-Tracker"
 				(path "/c19b4b11-d562-4619-8198-7fbe4f513d32/087e4c3f-dadb-4b00-b947-e0c7adeb7ff5"
 					(reference "#PWR01")
@@
 				)
 			)
-			(project ""
+			(project "TinyPico-Cycling-Tracker"
 				(path "/c19b4b11-d562-4619-8198-7fbe4f513d32/087e4c3f-dadb-4b00-b947-e0c7adeb7ff5"
 					(reference "U6")
@@
 				)
 			)
-			(project ""
+			(project "TinyPico-Cycling-Tracker"
 				(path "/c19b4b11-d562-4619-8198-7fbe4f513d32/087e4c3f-dadb-4b00-b947-e0c7adeb7ff5"
 					(reference "U7")
@@
 				)
 			)
-			(project ""
+			(project "TinyPico-Cycling-Tracker"
 				(path "/c19b4b11-d562-4619-8198-7fbe4f513d32/087e4c3f-dadb-4b00-b947-e0c7adeb7ff5"
 					(reference "R2")
@@
 				)
 			)
-			(project ""
+			(project "TinyPico-Cycling-Tracker"
 				(path "/c19b4b11-d562-4619-8198-7fbe4f513d32/087e4c3f-dadb-4b00-b947-e0c7adeb7ff5"
 					(reference "#PWR06")
@@
 				)
 			)
-			(project ""
+			(project "TinyPico-Cycling-Tracker"
 				(path "/c19b4b11-d562-4619-8198-7fbe4f513d32/087e4c3f-dadb-4b00-b947-e0c7adeb7ff5"
 					(reference "#FLG01")
